File: power-reset/asetniopy-power-reset.kicad_sch (KiCad schematic)
At the start: 5 parts, among them J1 Conn_01x03_Female, SW1 Reset, SW2 Power

Commit message: Add LSCS part numbers to power/reset.
Parts:
- SW1: LCSC Part Number (none) -> C79174
- SW2: LCSC Part Numbre (none) -> C221841
Changed lines of the file:
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@@
+      (effects (font (size 1.27 1.27)) hide)
+    )
+    (property "LCSC Part Number" "C79174" (id 4) (at 114.3 76.2 0)
       (effects (font (size 1.27 1.27)) hide)
     )
@@
       (effects (font (size 1.27 1.27)) hide)
     )
+    (property "LCSC Part Numbre" "C221841" (id 4) (at 163.83 73.025 0)
+      (effects (font (size 1.27 1.27)) hide)
+    )

Commit message: Fix property name typo.
Parts:
- SW2: LCSC Part Number (none) -> C221841; LCSC Part Numbre C221841 -> (none)
Changed lines of the file:
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@@
       (effects (font (size 1.27 1.27)) hide)
     )
-    (property "LCSC Part Numbre" "C221841" (id 4) (at 163.83 73.025 0)
+    (property "LCSC Part Number" "C221841" (id 4) (at 163.83 73.025 0)
       (effects (font (size 1.27 1.27)) hide)
     )
